File: Modules/SensorBug/v1/sensorbug_v1.sch (EAGLE design)
At the start: 43 parts, among them IC1 MX25R8035FZUIL0, T2 DMP3010LK3

Commit message: Fixed Light Sensor Output
Previous light sensor output pin did not have ADC capabilities.
Interchanged DOMAIN1_EN and LIGHT_OUT.
Connections:
- net DOMAIN1_EN: now also U$4.11; no longer U$4.13
- net LIGHT_OUT: now also U$4.13; no longer U$4.11
Changed lines of the file:
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@@
-</segment>
-<segment>
-<pinref part="U$4" gate="G$1" pin="13"/>
-<wire x1="-10.16" y1="10.16" x2="-17.78" y2="10.16" width="0.1524" layer="91"/>
-<label x="-25.4" y="10.16" size="1.778" layer="95"/>
 </segment>
 <segment>
@@
 <wire x1="228.6" y1="248.92" x2="220.98" y2="248.92" width="0.1524" layer="91"/>
 <label x="213.36" y="248.92" size="1.778" layer="95"/>
+</segment>
+<segment>
+<pinref part="U$4" gate="G$1" pin="11"/>
+<wire x1="-10.16" y1="12.7" x2="-17.78" y2="12.7" width="0.1524" layer="91"/>
+<label x="-25.4" y="12.7" size="1.778" layer="95"/>
 </segment>
 </net>
@@
 </segment>
 <segment>
-<pinref part="U$4" gate="G$1" pin="11"/>
-<wire x1="-10.16" y1="12.7" x2="-17.78" y2="12.7" width="0.1524" layer="91"/>
-<label x="-25.4" y="12.7" size="1.778" layer="95"/>
+<pinref part="U$4" gate="G$1" pin="13"/>
+<wire x1="-10.16" y1="10.16" x2="-17.78" y2="10.16" width="0.1524" layer="91"/>
+<label x="-25.4" y="10.16" size="1.778" layer="95"/>
 </segment>
 </net>
